File: compute-deck.kicad_pcb (KiCad board)
At the start: 4 copper layers, 70.5 x 88.9 mm, 63 parts, among them J1 USB_C_Receptacle_USB2.0_16P, J2 Conn_01x02, J3 Conn_01x02, J4 Conn_01x08, Q1 BSS138, SW1 SW_Push, U1 IP5306, U2 RP2040, U3 W25Q128JVS, U4 BBQ10KBD, Y1 12MHz

Commit message: add revision 2
Parts:
- removed FB1: 600R, Inductor_SMD:L_0603_1608Metric
- added Q2: Q_PMOS, Package_TO_SOT_SMD:SOT-23, B.Cu at (82.7, 92.1)
- added SW2: SW_SPDT, Button_Switch_SMD:SW_SPDT_PCM12, B.Cu at (34.3, 138.0)
- C1, C2, C3, C4, C5, C6, C8, J1, L1, R3, SW1, U1: moved to B.Cu
- C7: footprint Capacitor_SMD:C_0603_1608Metric -> Capacitor_SMD:C_0402_1005Metric; moved to B.Cu
- R1, R2, R4, R5: footprint Resistor_SMD:R_0603_1608Metric -> Resistor_SMD:R_0402_1005Metric; moved to B.Cu
- R11, R6, R7, R8, R9: footprint Resistor_SMD:R_0603_1608Metric -> Resistor_SMD:R_0402_1005Metric
- moved J3 54.3 mm to (26.8, 115.4)
- moved C20 27.2 mm to (62.2, 127.5), turned to 180 degrees
- moved R7 23.5 mm to (73.2, 116.0), turned to 90 degrees
- moved R8 21.1 mm to (63.0, 115.0), turned to -90 degrees
- moved U3 20.9 mm to (65.0, 121.2), turned to -90 degrees
- moved C12 20.2 mm to (78.5, 110.0), turned to 0 degrees
- moved R6 19.8 mm to (72.0, 116.0), turned to 90 degrees
- moved Y1 18.8 mm to (69.0, 99.0), turned to 0 degrees
- moved C14 18.7 mm to (78.5, 112.0), turned to 0 degrees
- moved R9 17.9 mm to (70.8, 103.0), turned to 90 degrees
- moved R11 16.6 mm to (61.2, 115.0)
- moved C16 15.7 mm to (70.8, 116.8), turned to -90 degrees
- moved C9 15.4 mm to (69.5, 116.8), turned to -90 degrees
- moved R5 14.4 mm to (38.6, 84.8), turned to 180 degrees
- moved C22 13.7 mm to (70.2, 101.5), turned to 0 degrees
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Connections:
- A1 pad 3: /KBD_SCL -> /KBD_SDA
- A1 pad 5: /KBD_SDA -> /KBD_SCL
- C8 pad 1: /BAT+ -> /CHRG_OUT
- J1 pad S1: /SHIELD -> GND
- J2 pad 1: /BAT+ -> GND
- J2 pad 2: GND -> /BAT+
- L1 pad 2: /BAT+ -> /CHRG_OUT
- R4 pad 1: /BAT+ -> /CHRG_OUT
- R6 pad 2: /D+ -> /RP2040 I2C Bridge/PI_D+
- R7 pad 2: /D- -> /RP2040 I2C Bridge/PI_D-
- U2 pad 17: unconnected-(U2-GPIO14-Pad17) -> /RP2040 I2C Bridge/BL_CONTROL
- U2 pad 29: unconnected-(U2-GPIO18-Pad29) -> /RP2040 I2C Bridge/A
- U2 pad 30: unconnected-(U2-GPIO19-Pad30) -> /RP2040 I2C Bridge/B
- U2 pad 31: unconnected-(U2-GPIO20-Pad31) -> /RP2040 I2C Bridge/C
- U2 pad 32: unconnected-(U2-GPIO21-Pad32) -> /RP2040 I2C Bridge/D
- U2 pad 34: unconnected-(U2-GPIO22-Pad34) -> /RP2040 I2C Bridge/CLICK
- U2 pad 46: /D- -> /RP2040 I2C Bridge/PI_D-
- U2 pad 47: /D+ -> /RP2040 I2C Bridge/PI_D+
Routing:
- net /ON: track 0.00 -> 86.5 mm
- net /BAT+: track 37.3 -> 92.8 mm, vias 0 -> 7
- net /VOUT: track 49.5 -> 4.02 mm, vias 0 -> 10
- net /RP2040 I2C Bridge/COL1: track 63.2 -> 28.6 mm, vias 2 -> 0
- net +1V1: track 9.17 -> 43.1 mm, vias 3 -> 2
- net /RP2040 I2C Bridge/COL2: track 60.9 -> 27.4 mm, vias 2 -> 0
- net /RP2040 I2C Bridge/~{USB_BOOT}: track 4.53 -> 37.2 mm
- net /RP2040 I2C Bridge/COL3: track 58.5 -> 26.0 mm, vias 2 -> 0
- net /RP2040 I2C Bridge/COL4: track 43.2 -> 17.2 mm, vias 2 -> 0
- net /BAT: track 7.75 -> 33.1 mm, vias 0 -> 2
- net /RP2040 I2C Bridge/BL_CONTROL: track 1.85 -> 26.9 mm
- net /RP2040 I2C Bridge/ROW3: track 41.7 -> 17.2 mm, vias 2 -> 0
- net /RP2040 I2C Bridge/ROW4: track 39.7 -> 17.0 mm, vias 2 -> 0
- net /RP2040 I2C Bridge/ROW5: track 39.2 -> 17.0 mm, vias 2 -> 0
- net /RP2040 I2C Bridge/ROW6: track 39.2 -> 19.2 mm, vias 2 -> 0
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- added copper zone on B.Cu, net /BAT+
- added copper zone on B.Cu, net /CHRG_OUT
- added copper zone on B.Cu, net /SW
- added copper zone on B.Cu, net /VBUS
- added copper zone on B.Cu, net /VOUT
- added copper zone on In2.Cu, net /VOUT
- removed copper zone on In2.Cu, net +1V1
- removed copper zone on F.Cu, net /SW
- removed copper zone on F.Cu, net /VOUT
Other:
- outline, holes or cut-outs redrawn
- board text added: "BOOTSEL"
- board text removed: "RST Jumper"
- board text removed: "Wake"
