File: compute-deck.kicad_sch (KiCad schematic)
At the start: 35 parts, among them J1 USB_C_Receptacle_USB2.0_16P, J2 Conn_01x02, J4 Conn_01x08, SW1 SW_Push, U1 IP5306

Commit message: add revision 2
Parts:
- removed FB1: 600R, Inductor_SMD:L_0603_1608Metric, symbol Device:FerriteBead_Small
- added Q2: Q_PMOS, Package_TO_SOT_SMD:SOT-23, symbol Device:Q_PMOS
- added SW2: SW_SPDT, Button_Switch_SMD:SW_SPDT_PCM12, symbol Switch:SW_SPDT
- C7: footprint Capacitor_SMD:C_0603_1608Metric -> Capacitor_SMD:C_0402_1005Metric
- R1, R2, R4, R5: footprint Resistor_SMD:R_0603_1608Metric -> Resistor_SMD:R_0402_1005Metric
Connections:
- net SHIELD is gone; now on net GND: J1.S1 (SHIELD)
- net BAT+: now also J2.2 (Pin_2), Q2.S, SW2.3 (C); no longer C8.1, J2.1 (Pin_1), L1.2, R4.1
- net GND: now also J2.1 (Pin_1), SW2.1 (A); no longer J2.2 (Pin_2)
- net KBD_SCL: now also A1.5 (GPIO3/SCL); no longer A1.3 (GPIO2/SDA)
- net KBD_SDA: now also A1.3 (GPIO2/SDA); no longer A1.5 (GPIO3/SCL)
- new net CHRG_OUT: C8.1, L1.2, Q2.D, R4.1
- new net ON: Q2.G, SW2.2 (B)
Other:
- note added: "Global ON/OFF switch"
- note added: "Recommended JLCPCB Stackup JLC04161H-3313A(Special/Finished thickness1.58mm±10%) This stackup does not support economic assembly. Not required since USB is only used for flashing the RP2040 firmware, but for careful impedance control pick this stackup."
