File: rp2040_i2c_bridge.kicad_sch (KiCad schematic)
At the start: 26 parts, among them J3 Conn_01x02, Q1 BSS138, U2 RP2040, U3 W25Q128JVS, U4 BBQ10KBD, Y1 12MHz

Commit message: add revision 2
Parts:
- R11, R6, R7, R8, R9: footprint Resistor_SMD:R_0603_1608Metric -> Resistor_SMD:R_0402_1005Metric
Connections:
- net BL_CONTROL: now also U2.17 (GPIO14)
- net USB_D+: no longer R6.2, U2.47 (USB_DP)
- net USB_D-: no longer R7.2, U2.46 (USB_DM)
- net A: now reaches U2.29 (GPIO18)
- net B: now reaches U2.30 (GPIO19)
- net C: now reaches U2.31 (GPIO20)
- net D: now reaches U2.32 (GPIO21)
- net CLICK: now reaches U2.34 (GPIO22)
- new net PI_D+: R6.2, U2.47 (USB_DP)
- new net PI_D-: R7.2, U2.46 (USB_DM)
- no-connect marks 20 -> 14
